File: kicad/floatController.kicad_pcb (KiCad board)
At the start: 4 copper layers, 101.6 x 91.4 mm, 134 parts, among them J1 Molex_KK156_2, J10 Molex_KK100_2, J11 FPC5, J12 Molex_KK100_5, J13 Hirose_DF11_2x2, J14 Hirose_DF11_2x2, J15 Molex_KK100_2, J17 JST_SH_4_Vert, J18 JST_SH_3_Vert, J2 Molex_KK100_4, J3 Molex_KK100_6, J4 Hirose_DF11_2x8, J5 Molex_KK100_6, J6 Molex_KK100_4, J7 PinSocket_2.54mm_4, J8 Molex_KK100_3, J9 Molex_KK100_2, Q1 DMN3023L-7, Q12 DMG6601LVT, Q2 SI4497, Q3 Si4554DY, Q4 Si4554DY, Q5 Si4554DY, Q6 Si4554DY, Q7 Si4554DY, Q8 Si4554DY, SW1 MS-106-3-x, U1 TEENSY_3.5_3.6, U10 LTC4311, U11 ESP-07, U12 TPS709xx, U13 TB67H451FNG, U14 TB67H451FNG, U15 TB67H451FNG, U16 TB67H451FNG, U17 BA06CC0WFP, U18 TB67H451FNG, U2 TINY25, U3 LMZM2360X, U4 TPSM842X, U5 INA233, U6 MAX3221, U7 MAX3221, U8 LSM9DS1, U9 BME280

Commit message: sync up
Parts:
- added MT5: MountingHole, MountingHole:MountingHole_2.5mm, F.Cu at (101.0, 86.1)
- added MT6: MountingHole, MountingHole:MountingHole_2.5mm, F.Cu at (126.0, 89.6)
- moved R20 2.77 mm to (122.0, 91.6)
- moved R22 2.75 mm to (126.3, 93.4)
Routing:
- net 12V_ENABLE: track 75.5 -> 79.6 mm
- net +BATT: track 318.1 -> 322.0 mm
- net PM_ALERT: track 46.7 -> 44.2 mm
- net DTR: track 38.9 -> 40.6 mm
- net RTS: track 39.3 -> 40.7 mm
- net CTS: track 36.0 -> 37.4 mm
- net DCD: track 39.8 -> 41.0 mm
- net SDA1: track 73.0 -> 72.3 mm
- net SERCTL3: track 68.8 -> 68.1 mm
- net NETAVAIL: track 36.3 -> 35.7 mm
- net SCK2: track 30.8 -> 31.4 mm
