File: kicad/floatController.sch (KiCad schematic (older format))
At the start: 15 parts, among them J18 JST_SH_3_Vert, J8 Molex_KK100_3, U1 TEENSY_3.5_3.6, U11 ESP-07

Commit message: sync up
Parts:
- added MT5, MT6: MountingHole, MountingHole:MountingHole_2.5mm, symbol Mechanical:MountingHole
Changed lines of the file:
@@
+	1    0    0    -1
+$EndComp
+$Comp
+L Mechanical:MountingHole MT5
+U 1 1 60656C4F
+P 950 9665
+F 0 "MT5" H 1050 9711 50  0000 L CNN
+F 1 "MountingHole" H 1050 9620 50  0000 L CNN
+F 2 "MountingHole:MountingHole_2.5mm" H 950 9665 50  0001 C CNN
+F 3 "~" H 950 9665 50  0001 C CNN
+	1    950  9665
+	1    0    0    -1
+$EndComp
+$Comp
+L Mechanical:MountingHole MT6
+U 1 1 60656FE9
+P 960 9910
+F 0 "MT6" H 1060 9956 50  0000 L CNN
+F 1 "MountingHole" H 1060 9865 50  0000 L CNN
+F 2 "MountingHole:MountingHole_2.5mm" H 960 9910 50  0001 C CNN
+F 3 "~" H 960 9910 50  0001 C CNN
+	1    960  9910
 	1    0    0    -1
 $EndComp
